File: knott/knott.kicad_sch (KiCad schematic)
At the start: 18 parts, among them SW1 SW_PUSH, SW10 SW_PUSH, SW11 SW_PUSH, SW12 SW_PUSH, SW13 SW_PUSH, SW14 SW_PUSH, SW15 SW_PUSH, SW2 SW_PUSH, SW3 SW_PUSH, SW4 SW_PUSH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

Commit message: Moved libraries into base directory.
Parts:
- BT1: footprint knott:Battery_pads_reversible -> bugs:Battery_pads_reversible
- PSW1: footprint knott:Power_reversible -> bugs:Power_reversible
- SW1: footprint knott:Choc_reversible -> bugs:Choc_reversible; symbol knott:SW_PUSH-kbd -> bugs:SW_PUSH-kbd
- SW10, SW11, SW12, SW13, SW14, SW15, SW2, SW3, SW4, SW5, SW6, SW7, SW8, SW9: footprint knott:Choc_reversible -> bugs:Choc_reversible
- U1: footprint knott:ProMicro_reversible -> bugs:ProMicro_reversible; symbol knott:ProMicro-kbd -> bugs:ProMicro-kbd
