File: locust/locust.kicad_sch (KiCad schematic)
At the start: 19 parts, among them SW1 SW_PUSH, SW10 SW_PUSH, SW11 SW_PUSH, SW12 SW_PUSH, SW13 SW_PUSH, SW14 SW_PUSH, SW15 SW_PUSH, SW16 SW_PUSH, SW2 SW_PUSH, SW3 SW_PUSH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

Commit message: Renamed Cicada to Locust.
Other:
- title: Cicada -> Locust
Changed lines of the file:
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@@
   (paper "A4")
   (title_block
-    (title "Cicada")
-    (date "2021-10-04")
-    (rev "0.1")
+    (title "Locust")
+    (date "2021-10-11")
+    (rev "0.2")
     (company "jmnw")
   )
