File: wasp/wasp.kicad_pcb (KiCad board)
At the start: 2 copper layers, 129 x 84.2 mm, 23 parts, among them SW1 SW_PUSH, SW10 SW_PUSH, SW11 SW_PUSH, SW12 SW_PUSH, SW13 SW_PUSH, SW14 SW_PUSH, SW15 SW_PUSH, SW16 SW_PUSH, SW17 SW_PUSH, SW2 SW_PUSH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

Commit message: Fixed a couple of traces.
Routing:
- net GND: track 49.9 -> 48.2 mm
Other:
- board text added: "Wasp v0.1.1 https://github.com/jimmerricks/bugs"
- board text removed: "Wasp v0.1 https://github.com/jimmerricks/bugs"
Changed lines of the file:
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@@
     (title "Wasp")
     (date "2021-10-11")
-    (rev "0.1")
+    (rev "0.1.1")
     (company "jmnw")
   )
@@
   (gr_line (start 139.336399 45.280745) (end 139.310739 54.770533) (layer "Edge.Cuts") (width 0.15))
   (gr_arc (start 141.310739 54.770531) (end 139.310739 54.770533) (angle -90) (layer "Edge.Cuts") (width 0.15))
-  (gr_text "Wasp v0.1\nhttps://github.com/jimmerricks/bugs" (at 149.94 66.220003 90) (layer "B.SilkS")
+  (gr_text "Wasp v0.1.1\nhttps://github.com/jimmerricks/bugs" (at 149.94 66.220003 90) (layer "B.SilkS")
     (effects (font (size 0.8 0.8) (thickness 0.1)) (justify left mirror))
   )
-  (gr_text "Wasp v0.1\nhttps://github.com/jimmerricks/bugs" (at 149.94 89.44 90) (layer "F.SilkS")
+  (gr_text "Wasp v0.1.1\nhttps://github.com/jimmerricks/bugs" (at 149.94 89.44 90) (layer "F.SilkS")
     (effects (font (size 0.8 0.8) (thickness 0.1)) (justify left))
   )
@@
   (segment (start 152.856544 86.436591) (end 153.052201 86.240932) (width 0.25) (layer "B.Cu") (net 9))
   (arc (start 151.795877 86.875937) (mid 152.369907 86.761755) (end 152.856544 86.436591) (width 0.25) (layer "B.Cu") (net 9))
-  (segment (start 106.236209 75.512337) (end 106.236209 69.430931) (width 0.25) (layer "F.Cu") (net 10))
-  (segment (start 106.236204 75.512342) (end 106.236209 75.512337) (width 0.25) (layer "F.Cu") (net 10))
   (segment (start 143.7652 83.700934) (end 144.400198 84.335933) (width 0.25) (layer "F.Cu") (net 10))
   (segment (start 143.400201 83.700935) (end 142.584381 82.885115) (width 0.25) (layer "F.Cu") (net 10))
+  (segment (start 106.236209 69.430931) (end 106.236209 74.269705) (width 0.25) (layer "F.Cu") (net 10))
   (segment (start 141.523721 82.445776) (end 136.754121 82.445777) (width 0.25) (layer "F.Cu") (net 10))
+  (segment (start 107.114889 76.391026) (end 108.557338 77.833475) (width 0.25) (layer "F.Cu") (net 10))
   (segment (start 106.236211 69.430928) (end 116.436206 69.430925) (width 0.25) (layer "F.Cu") (net 10))
-  (segment (start 106.236204 75.512342) (end 108.557338 77.833475) (width 0.25) (layer "F.Cu") (net 10))
   (segment (start 131.156537 78.712155) (end 110.678658 78.712155) (width 0.25) (layer "F.Cu") (net 10))
   (segment (start 135.693461 82.006437) (end 133.277857 79.590834) (width 0.25) (layer "F.Cu") (net 10))
@@
   (arc (start 135.693461 82.006437) (mid 136.180096 82.331596) (end 136.754121 82.445777) (width 0.25) (layer "F.Cu") (net 10))
   (arc (start 141.523721 82.445776) (mid 142.097746 82.559957) (end 142.584381 82.885115) (width 0.25) (layer "F.Cu") (net 10))
+  (arc (start 106.236209 74.269705) (mid 106.464571 75.417756) (end 107.114889 76.391026) (width 0.25) (layer "F.Cu") (net 10))
   (arc (start 108.557338 77.833475) (mid 109.530608 78.483793) (end 110.678658 78.712155) (width 0.25) (layer "F.Cu") (net 10))
   (segment (start 152.85654 83.896596) (end 153.052201 83.700935) (width 0.25) (layer "B.Cu") (net 10))
@@
   (segment (start 144.900199 65.920935) (end 143.400201 65.920935) (width 0.4) (layer "B.Cu") (net 20))
   (segment (start 152.351712 64.081419) (end 152.351711 66.891424) (width 0.4) (layer "B.Cu") (net 20))
-  (segment (start 135.663149 64.655776) (end 143.635042 64.655781) (width 0.4) (layer "B.Cu") (net 20))
   (segment (start 146.166774 66.56619) (end 150.806138 66.566191) (width 0.4) (layer "B.Cu") (net 20))
   (segment (start 152.351711 66.891424) (end 152.0522 67.190931) (width 0.4) (layer "B.Cu") (net 20))
   (segment (start 151.866795 67.005527) (end 152.0522 67.190931) (width 0.4) (layer "B.Cu") (net 20))
+  (segment (start 136.284469 64.655776) (end 141.513721 64.655776) (width 0.4) (layer "B.Cu") (net 20))
   (segment (start 143.400201 65.920935) (end 143.400203 68.460935) (width 0.4) (layer "B.Cu") (net 20))
   (segment (start 153.052197 63.380936) (end 152.351712 64.081419) (width 0.4) (layer "B.Cu") (net 20))
   (segment (start 148.984684 60.697745) (end 148.984682 60.297745) (width 0.4) (layer "B.Cu") (net 20))
-  (segment (start 143.635042 64.655781) (end 144.900199 65.920935) (width 0.4) (layer "B.Cu") (net 20))
-  (segment (start 129.688306 58.680933) (end 135.663149 64.655776) (width 0.4) (layer "B.Cu") (net 20))
+  (segment (start 142.574381 65.095116) (end 143.400199 65.920934) (width 0.4) (layer "B.Cu") (net 20))
+  (segment (start 129.688306 58.680933) (end 135.22381 64.216437) (width 0.4) (layer "B.Cu") (net 20))
   (segment (start 129.3362 58.680931) (end 129.688306 58.680933) (width 0.4) (layer "B.Cu") (net 20))
   (arc (start 145.106114 66.12685) (mid 145.592749 66.452009) (end 146.166774 66.56619) (width 0.4) (layer "B.Cu") (net 20))
+  (arc (start 141.513721 64.655776) (mid 142.087746 64.769957) (end 142.574381 65.095116) (width 0.4) (layer "B.Cu") (net 20))
+  (arc (start 135.22381 64.216437) (mid 135.710445 64.541596) (end 136.284469 64.655776) (width 0.4) (layer "B.Cu") (net 20))
   (arc (start 151.866795 67.005527) (mid 151.380161 66.68037) (end 150.806138 66.566191) (width 0.4) (layer "B.Cu") (net 20))
   (segment (start 143.400201 68.730932) (end 144.400201 69.730933) (width 0.4) (layer "F.Cu") (net 21))
