File: termite/termite.kicad_pcb (KiCad board)
At the start: 2 copper layers, 119.7 x 84.2 mm, 19 parts, among them SW1 SW_PUSH, SW10 SW_PUSH, SW11 SW_PUSH, SW12 SW_PUSH, SW13 SW_PUSH, SW14 SW_PUSH, SW15 SW_PUSH, SW16 SW_PUSH, SW2 SW_PUSH, SW3 SW_PUSH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

Commit message: Renamed Locust to Termite and changed the battery footprint.
Parts:
- BT1: footprint bugs:Battery_holes -> bugs:Battery_pads_reversible
Routing:
- net Net-(BT1-Pad2): track 40.5 -> 40.4 mm, vias 1 -> 2
- net raw: vias 2 -> 3
Other:
- board text added: "Termite v0.2.1 https://github.com/jimmerricks/bugs"
- board text removed: "Locust v0.1 https://github.com/jimmerricks/bugs"
- board text removed: "Locust v0.2 https://github.com/jimmerricks/bugs"
Changed lines of the file:
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@@
   (paper "A4")
   (title_block
-    (title "Cicada")
-    (date "2021-10-04")
-    (rev "0.1")
+    (title "Termite")
+    (date "2021-10-28")
+    (rev "0.2.1")
     (company "jmnw")
   )
@@
       (layer "F.SilkS" (type "Top Silk Screen") (color "White"))
       (layer "F.Paste" (type "Top Solder Paste"))
-      (layer "F.Mask" (type "Top Solder Mask") (color "Green") (thickness 0.01))
+      (layer "F.Mask" (type "Top Solder Mask") (color "Purple") (thickness 0.01))
       (layer "F.Cu" (type "copper") (thickness 0.035))
       (layer "dielectric 1" (type "core") (thickness 1.51) (material "FR4") (epsilon_r 4.5) (loss_tangent 0.02))
       (layer "B.Cu" (type "copper") (thickness 0.035))
-      (layer "B.Mask" (type "Bottom Solder Mask") (color "Green") (thickness 0.01))
+      (layer "B.Mask" (type "Bottom Solder Mask") (color "Purple") (thickness 0.01))
       (layer "B.Paste" (type "Bottom Solder Paste"))
       (layer "B.SilkS" (type "Bottom Silk Screen") (color "White"))
@@
       (net 19 "GND") (pinfunction "2"))
   )
-  (footprint "bugs:Battery_holes" (layer "F.Cu")
+  (footprint "bugs:Battery_pads_reversible" (layer "F.Cu")
     (at 133.062606 100.452098 180)
     (property "Sheetfile" "cicada.kicad_sch")
     (property "Sheetname" "")
-    (fp_text reference "BT1" (at -0.2 0.3) (layer "F.SilkS") hide
+    (fp_text reference "BT1" (at 0 0.5 180) (layer "F.SilkS") hide
       (effects (font (size 1 1) (thickness 0.15)))
     )
-    (fp_text value "Battery_Cell" (at 0 -4.1) (layer "F.Fab")
+    (fp_text value "Battery_Cell" (at 0 -0.5 180) (layer "F.Fab")
       (effects (font (size 1 1) (thickness 0.15)))
     )
+    (fp_text user "Battery" (at 0 -2.2) (layer "B.SilkS") hide
+      (effects (font (size 1 1) (thickness 0.12)) (justify mirror))
+    )
     (fp_text user "BT01" (at 0 0.5) (layer "B.SilkS") hide
       (effects (font (size 1 1) (thickness 0.15)) (justify mirror))
     )
-    (fp_text user "(-)" (at 1.28825 -2.22825) (layer "B.SilkS") hide
-      (effects (font (size 0.8 0.8) (thickness 0.1)) (justify mirror))
-    )
-    (fp_text user "(+)" (at -1.31175 -2.22825) (layer "B.SilkS") hide
-      (effects (font (size 0.8 0.8) (thickness 0.1)) (justify mirror))
+    (fp_text user "(-)" (at 1.1 -2.032) (layer "B.SilkS")
+      (effects (font (size 0.8 0.8) (thickness 0.12)) (justify mirror))
     )
-    (fp_text user "Battery" (at 3.35 -0.87825 90) (layer "B.SilkS") hide
-      (effects (font (size 0.8 0.8) (thickness 0.1)) (justify mirror))
+    (fp_text user "(+)" (at -1.1 -2.032) (layer "B.SilkS")
+      (effects (font (size 0.8 0.8) (thickness 0.12)) (justify mirror))
     )
-    (fp_text user "Battery" (at 3.35 -0.87825 90) (layer "F.SilkS") hide
-      (effects (font (size 0.8 0.8) (thickness 0.1)))
+    (fp_text user "Battery" (at 0 -2.2 180) (layer "F.SilkS") hide
+      (effects (font (size 1 1) (thickness 0.12)))
     )
-    (fp_text user "(-)" (at 1.28825 -2.22825) (layer "F.SilkS") hide
-      (effects (font (size 0.8 0.8) (thickness 0.1)))
+    (fp_text user "(+)" (at -1.1 -2.032 180) (layer "F.SilkS")
+      (effects (font (size 0.8 0.8) (thickness 0.12)))
     )
-    (fp_text user "(+)" (at -1.31175 -2.22825) (layer "F.SilkS") hide
-      (effects (font (size 0.8 0.8) (thickness 0.1)))
+    (fp_text user "(-)" (at 1.1 -2.032 180) (layer "F.SilkS")
+      (effects (font (size 0.8 0.8) (thickness 0.12)))
     )
-    (fp_text user "Battery_Cell" (at 0 -4.1) (layer "B.Fab")
+    (fp_text user "Battery_Cell" (at 0 -0.5) (layer "B.Fab")
       (effects (font (size 1 1) (thickness 0.15)) (justify mirror))
     )
-    (pad "1" thru_hole circle (at -1.3 0 180) (size 1.8 1.8) (drill 1.2) (layers *.Cu *.Mask)
+    (fp_poly (pts
+        (xy 1.8 1)
+        (xy 1.8 -1)
+        (xy 0.4 -1)
+        (xy 0.4 1)
+      ) (layer "B.Mask") (width 0.1) (fill solid))
+    (fp_poly (pts
+        (xy -0.4 1)
+        (xy -0.4 -1)
+        (xy -1.8 -1)
+        (xy -1.8 1)
+      ) (layer "B.Mask") (width 0.1) (fill solid))
+    (fp_poly (pts
+        (xy -1.798558 1)
+        (xy -1.798558 -1)
+        (xy -0.398558 -1)
+        (xy -0.398558 1)
+      ) (layer "F.Mask") (width 0.1) (fill solid))
+    (fp_poly (pts
+        (xy 0.4 1)
+        (xy 0.4 -1)
+        (xy 1.8 -1)
+        (xy 1.8 1)
+      ) (layer "F.Mask") (width 0.1) (fill solid))
+    (pad "1" smd rect (at -1.1 0 180) (size 1.5 2.1) (layers "F.Cu")
+      (net 22 "raw") (pinfunction "+"))
+    (pad "1" smd rect (at -1.1 0) (size 1.5 2.1) (layers "B.Cu")
       (net 22 "raw") (pinfunction "+"))
-    (pad "2" thru_hole rect (at 1.3 0 180) (size 1.8 2) (drill 1.2) (layers *.Cu *.Mask)
+    (pad "2" smd rect (at 1.1 0) (size 1.5 2.1) (layers "B.Cu")
+      (net 21 "Net-(BT1-Pad2)") (pinfunction "-"))
+    (pad "2" smd rect (at 1.1 0 180) (size 1.5 2.1) (layers "F.Cu")
       (net 21 "Net-(BT1-Pad2)") (pinfunction "-"))
   )
@@
   (gr_line (start 130.495061 53.956158) (end 130.469401 63.445945) (layer "Edge.Cuts") (width 0.15))
   (gr_arc (start 132.469403 63.445942) (end 130.469401 63.445945) (angle -90) (layer "Edge.Cuts") (width 0.15))
-  (gr_text "Locust v0.1\nhttps://github.com/jimmerricks/bugs" (at 141.170001 74.890001 90) (layer "B.SilkS")
+  (gr_text "Termite v0.2.1\nhttps://github.com/jimmerricks/bugs" (at 141.170001 74.890001 90) (layer "B.SilkS")
     (effects (font (size 0.8 0.8) (thickness 0.1)) (justify left mirror))
   )
-  (gr_text "Locust v0.2\nhttps://github.com/jimmerricks/bugs" (at 141.17 98.11 90) (layer "F.SilkS")
+  (gr_text "Termite v0.2.1\nhttps://github.com/jimmerricks/bugs" (at 141.17 98.11 90) (layer "F.SilkS")
     (effects (font (size 0.8 0.8) (thickness 0.1)) (justify left))
   )
@@
   (arc (start 135.826928 78.241835) (mid 135.731258 78.260864) (end 135.650154 78.315056) (width 0.4) (layer "B.Cu") (net 20))
   (arc (start 142.691161 78.241834) (mid 143.07384 78.165712) (end 143.398265 77.948941) (width 0.4) (layer "B.Cu") (net 20))
-  (segment (start 141.643342 69.373156) (end 141.643342 70.067878) (width 0.25) (layer "F.Cu") (net 21))
+  (segment (start 137.162054 74.549165) (end 140.665027 71.046189) (width 0.25) (layer "F.Cu") (net 21))
   (segment (start 135.999055 98.695651) (end 136.136931 98.557776) (width 0.25) (layer "F.Cu") (net 21))
+  (segment (start 131.962606 100.452098) (end 131.962606 100.252098) (width 0.25) (layer "F.Cu") (net 21))
+  (segment (start 133.786819 98.842099) (end 134.201034 98.842099) (width 0.25) (layer "F.Cu") (net 21))
+  (segment (start 141.643342 69.373156) (end 141.643342 70.067878) (width 0.25) (layer "F.Cu") (net 21))
+  (segment (start 131.962606 100.252098) (end 133.079712 99.134992) (width 0.25) (layer "F.Cu") (net 21))
+  (segment (start 134.201034 98.842099) (end 135.6455 98.842097) (width 0.25) (layer "F.Cu") (net 21))
   (segment (start 141.643342 70.067878) (end 140.665027 71.046189) (width 0.25) (layer "F.Cu") (net 21))
   (segment (start 136.283376 98.204224) (end 136.283375 76.670483) (width 0.25) (layer "F.Cu") (net 21))
-  (segment (start 137.162054 74.549165) (end 140.665027 71.046189) (width 0.25) (layer "F.Cu") (net 21))
-  (segment (start 134.201034 98.842099) (end 135.6455 98.842097) (width 0.25) (layer "F.Cu") (net 21))
-  (segment (start 131.762607 100.452098) (end 132.786821 99.427883) (width 0.25) (layer "F.Cu") (net 21))
   (via (at 140.665027 71.046189) (size 0.8) (drill 0.4) (layers "F.Cu" "B.Cu") (net 21))
-  (arc (start 136.283376 98.204224) (mid 136.245315 98.395562) (end 136.136931 98.557776) (width 0.25) (layer "F.Cu") (net 21))
-  (arc (start 134.201034 98.842099) (mid 133.435667 98.994339) (end 132.786821 99.427883) (width 0.25) (layer "F.Cu") (net 21))
+  (via (at 131.962606 100.452098) (size 0.8) (drill 0.4) (layers "F.Cu" "B.Cu") (net 21))
   (arc (start 136.283375 76.670483) (mid 136.511737 75.522433) (end 137.162054 74.549165) (width 0.25) (layer "F.Cu") (net 21))
+  (arc (start 136.136931 98.557776) (mid 136.245315 98.395562) (end 136.283376 98.204224) (width 0.25) (layer "F.Cu") (net 21))
+  (arc (start 133.079712 99.134992) (mid 133.404135 98.918219) (end 133.786819 98.842099) (width 0.25) (layer "F.Cu") (net 21))
   (arc (start 135.6455 98.842097) (mid 135.836842 98.804036) (end 135.999055 98.695651) (width 0.25) (layer "F.Cu") (net 21))
   (segment (start 137.143343 69.373155) (end 138.230589 70.460401) (width 0.25) (layer "B.Cu") (net 21))
@@
   (via (at 136.558865 72.691345) (size 0.8) (drill 0.4) (layers "F.Cu" "B.Cu") (net 22))
   (via (at 140.064696 72.855853) (size 0.8) (drill 0.4) (layers "F.Cu" "B.Cu") (net 22))
+  (via (at 134.162606 100.452098) (size 0.8) (drill 0.4) (layers "F.Cu" "B.Cu") (net 22))
   (arc (start 135.9855 100.159205) (mid 135.661077 100.375977) (end 135.278395 100.452097) (width 0.4) (layer "F.Cu") (net 22))
   (arc (start 134.851758 70.984239) (mid 134.634986 70.659816) (end 134.558864 70.277133) (width 0.4) (layer "F.Cu") (net 22))
