File: termite/termite.kicad_sch (KiCad schematic)
At the start: 19 parts, among them SW1 SW_PUSH, SW10 SW_PUSH, SW11 SW_PUSH, SW12 SW_PUSH, SW13 SW_PUSH, SW14 SW_PUSH, SW15 SW_PUSH, SW16 SW_PUSH, SW2 SW_PUSH, SW3 SW_PUSH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

Commit message: Renamed Locust to Termite and changed the battery footprint.
Other:
- title: Locust -> Termite
Changed lines of the file:
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@@
   (paper "A4")
   (title_block
-    (title "Locust")
-    (date "2021-10-11")
-    (rev "0.2")
+    (title "Termite")
+    (date "2021-10-28")
+    (rev "0.2.1")
     (company "jmnw")
   )
