File: pcbs/yellowjacket/yellowjacket.kicad_pcb (KiCad board)
At the start: 2 copper layers, 115 x 84.2 mm, 22 parts, among them SW1 SW_PUSH, SW10 SW_PUSH, SW11 SW_PUSH, SW12 SW_PUSH, SW13 SW_PUSH, SW14 SW_PUSH, SW15 SW_PUSH, SW16 SW_PUSH, SW2 SW_PUSH, SW3 SW_PUSH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

Commit message: Moved the pcbs into a subdirectory to tidy things up a little.
Routing:
- removed copper zone on F.Cu, net GND
Changed lines of the file:
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@@
   (segment (start 152.052203 88.145933) (end 144.656517 88.145935) (width 0.25) (layer "B.Cu") (net 24))
   (arc (start 143.595864 88.585267) (mid 144.082497 88.260113) (end 144.656517 88.145935) (width 0.25) (layer "B.Cu") (net 24))
-  (zone (net 20) (net_name "GND") (layers F&B.Cu) (hatch edge 0.508)
+  (zone (net 20) (net_name "GND") (layer "B.Cu") (hatch edge 0.508)
     (connect_pads (clearance 0.508))
     (min_thickness 0.254) (filled_areas_thickness no)

Commit message: Minor change and version bump for consistency with the Wasp.
Other:
- board text added: "Yellowjacket v0.1.2 https://github.com/jimmerricks/bugs"
- board text removed: "Yellowjacket v0.1.1 https://github.com/jimmerricks/bugs"
Changed lines of the file:
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@@
   (title_block
     (title "Yellowjacket")
-    (date "2021-10-28")
-    (rev "0.1.1")
+    (date "2021-10-31")
+    (rev "0.1.2")
     (company "jmnw")
   )
@@
       (drillshape 0)
       (scaleselection 1)
-      (outputdirectory "../gerbers/")
+      (outputdirectory "../../gerbers/")
     )
   )
@@
   (gr_line (start 139.336399 45.280745) (end 139.310739 54.770533) (layer "Edge.Cuts") (width 0.15))
   (gr_arc (start 141.310739 54.770531) (end 139.310739 54.770533) (angle -90) (layer "Edge.Cuts") (width 0.15))
-  (gr_text "Yellowjacket v0.1.1\nhttps://github.com/jimmerricks/bugs" (at 149.94 66.220003 90) (layer "B.SilkS")
+  (gr_text "Yellowjacket v0.1.2\nhttps://github.com/jimmerricks/bugs" (at 149.94 66.220003 90) (layer "B.SilkS")
     (effects (font (size 0.8 0.8) (thickness 0.1)) (justify left mirror))
   )
-  (gr_text "Yellowjacket v0.1.1\nhttps://github.com/jimmerricks/bugs" (at 149.94 89.44 90) (layer "F.SilkS")
+  (gr_text "Yellowjacket v0.1.2\nhttps://github.com/jimmerricks/bugs" (at 149.94 89.44 90) (layer "F.SilkS")
     (effects (font (size 0.8 0.8) (thickness 0.1)) (justify left))
   )
