File: pcbs/mosquito/mosquito.kicad_pcb (KiCad board)
At the start: 2 copper layers, 131.4 x 84.2 mm, 23 parts, among them SW1 SW_PUSH, SW10 SW_PUSH, SW11 SW_PUSH, SW12 SW_PUSH, SW13 SW_PUSH, SW14 SW_PUSH, SW15 SW_PUSH, SW16 SW_PUSH, SW17 SW_PUSH, SW2 SW_PUSH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

Commit message: Modified the silkscreen on the Mosquito.
Other:
- board text added: "Mosquito v0.1.1 https://github.com/jimmerricks/bugs"
- board text removed: "Mosquito v0.1 https://github.com/jimmerricks/bugs"
