File: pcbs/flea/flea.kicad_sch (KiCad schematic)
At the start: 18 parts, among them SW1 SW_PUSH, SW10 SW_PUSH, SW11 SW_PUSH, SW12 SW_PUSH, SW13 SW_PUSH, SW14 SW_PUSH, SW15 SW_PUSH, SW2 SW_PUSH, SW3 SW_PUSH, SW4 SW_PUSH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

Commit message: Minor edits
Connections:
- net switch1: now also SW2.1; no longer SW1.1
- net switch10: now also SW1.1; no longer SW10.1
- net switch2: now also SW3.1; no longer SW2.1
- net switch3: now also SW4.1; no longer SW3.1
- net switch4: now also SW5.1; no longer SW4.1
- net switch5: now also SW6.1; no longer SW5.1
- net switch6: now also SW7.1; no longer SW6.1
- net switch7: now also SW8.1; no longer SW7.1
- net switch8: now also SW9.1; no longer SW8.1
- net switch9: now also SW10.1; no longer SW9.1
Other:
- moved on the sheet: SW1
